File: fujinet-devkit-shield.kicad_pcb (KiCad board)
At the start: 2 copper layers, 92.7 x 55.9 mm, 42 parts, among them J1 SIO (No 12V), J2 Conn_BUTTON_A, J3 SD BOARD, J4 Conn_BUTTON_B, J5 Conn_BUTTON_RESET, J6 Conn_WHITE_LED, J7 Conn_ORANGE_LED, J8 Conn_BLUE_LED, P1 ST-TF-003A, SW1 BUTTON A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

Commit message: Files sent to JCL
Parts:
- added C5: 10uf 6.3V, Capacitor_THT:CP_Radial_D5.0mm_P2.00mm, F.Cu at (117.5, 110.0)
- added D4: 1N5817, Diode_THT:D_DO-41_SOD81_P10.16mm_Horizontal, F.Cu at (130.8, 81.3)
- added J10: DB15_Female_MountingHoles, Connector_Dsub:DSUB-15_Female_Horizontal_P2.77x2.84mm_EdgePinOffset7.70mm_Housed_MountingHolesOffset9.12mm, F.Cu at (111.8, 94.7)
- added REF**: KiCad-Logo2_5mm_SilkScreen, Symbol:KiCad-Logo2_5mm_SilkScreen, F.Cu at (163.1, 101.6)
- added REF**: OSHW-Logo_5.7x6mm_SilkScreen, Symbol:OSHW-Logo_5.7x6mm_SilkScreen, F.Cu at (151.1, 101.6)
- C1: footprint Capacitor_THT:CP_Radial_D5.0mm_P2.50mm -> Capacitor_THT:C_Rect_L7.0mm_W3.5mm_P2.50mm_P5.00mm
- C4: value 10uF 25V -> 10uF 6.3V
- J1: footprint Connector_PinHeader_2.54mm:PinHeader_1x12_P2.54mm_Horizontal -> Connector_PinHeader_2.54mm:PinHeader_1x12_P2.54mm_Vertical
- R9: value 1K -> 10K
- U1: value ESP32-DEVKITC-32U -> ESP32-DEVKITC-VE
- moved H1 8.62 mm to (107.6, 109.6)
- moved H2 8.62 mm to (107.6, 60.6)
- moved R10 6.35 mm to (122.7, 58.7)
- moved R11 6.10 mm to (122.7, 61.2)
- moved C1 5.94 mm to (120.9, 77.6)
- moved R12 5.84 mm to (122.7, 63.8)
- moved R13 5.59 mm to (122.7, 66.3)
- moved C4 4.58 mm to (121.2, 70.6), turned to 180 degrees
- moved H3 2.83 mm to (199.7, 109.6)
- moved H4 2.83 mm to (199.7, 60.6)
- moved D1 1.27 mm to (189.2, 102.2)
- moved D2 1.27 mm to (189.2, 69.8)
- moved D3 1.27 mm to (189.2, 88.9)
- moved J2 1.27 mm to (200.2, 94.5)
- moved J4 1.27 mm to (200.2, 81.3)
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Connections:
- J1 pad 10: +5V -> SIO_5V
Routing:
- net SIO_5V: track 0.00 -> 21.1 mm
- net +5V: track 112.8 -> 128.6 mm
- net SIO_MCTL: track 71.3 -> 85.7 mm
- net SIO_CMD: track 12.2 -> 26.4 mm
- net SIO_DATAOUT: track 24.1 -> 37.8 mm
- net SIO_PROC: track 35.0 -> 48.6 mm
- net SIO_CKIN: track 25.2 -> 37.9 mm
- net SIO_CKOUT: track 23.7 -> 35.9 mm
- net SIO_DATAIN: track 31.4 -> 42.7 mm
- net SIO_INT: track 31.9 -> 43.0 mm, vias 3 -> 1
- net SIO_AUDIOIN: track 8.74 -> 19.0 mm
- net Net-(C1-Pad2): track 3.85 -> 10.1 mm
- net +3V3: track 175.0 -> 171.7 mm
- net IO19_SPI_MISO: track 59.8 -> 62.4 mm
- net IO23_SPI_MOSI: track 63.5 -> 65.9 mm
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Other:
- board size 92.7 x 55.9 mm -> 99.1 x 55.9 mm
- board text added: "JLCJLCJLCJLC"

Commit message: First pass at some docs
Parts:
- C4: value 10uF 6.3V -> 10uF 10V
- H1, H2, H3, H4: value MountingHole -> M3 Mounting Hole
