File: fujinet-devkit-shield.sch (KiCad schematic (older format))
At the start: 42 parts, among them J1 SIO (No 12V), J2 Conn_BUTTON_A, J3 SD BOARD, J4 Conn_BUTTON_B, J5 Conn_BUTTON_RESET, J6 Conn_WHITE_LED, J7 Conn_ORANGE_LED, J8 Conn_BLUE_LED, P1 ST-TF-003A, SW1 BUTTON A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

Commit message: Files sent to JCL
Parts:
- added C5: 10uf 6.3V, Capacitor_THT:CP_Radial_D6.3mm_P2.50mm, symbol Device:CP1
- added D4: 1N5817, Diode_THT:D_DO-41_SOD81_P10.16mm_Horizontal, symbol Diode:1N5817
- added J10: DB15_Female_MountingHoles, Connector_Dsub:DSUB-15_Female_Horizontal_P2.77x2.84mm_EdgePinOffset4.94mm_Housed_MountingHolesOffset7.48mm, symbol Connector:DB15_Female_MountingHoles
- C1: footprint Capacitor_THT:CP_Radial_D5.0mm_P2.50mm -> Capacitor_THT:C_Disc_D5.1mm_W3.2mm_P5.00mm; symbol Device:CP1 -> Device:C
- J1: footprint Connector_PinHeader_2.54mm:PinHeader_1x12_P2.54mm_Horizontal -> Connector_PinHeader_2.54mm:PinHeader_1x12_P2.54mm_Vertical
- R9: value 1K -> 10K
- U1: value ESP32-DEVKITC-32U -> ESP32-DEVKITC-VE
Connections:
- net +5V: now also C5.1, D4.1 (K); no longer J1.10 (Pin_10)
- net GND: now also C5.2, J10.4, J10.6
- net SIO_AUDIOIN: now also J10.11 (P111)
- net SIO_CKIN: now also J10.1
- net SIO_CKOUT: now also J10.2
- net SIO_CMD: now also J10.7
- net SIO_DATAIN: now also J10.3
- net SIO_DATAOUT: now also J10.5
- net SIO_INT: now also J10.13 (P13)
- net SIO_MCTL: now also J10.8
- net SIO_PROC: now also J10.9 (P9)
- new net SIO_5V: D4.2 (A), J1.10 (Pin_10), J10.10 (P10)
- no-connect marks 0 -> 1
Other:
- moved on the sheet: C2, C3, H1, H2, H3, H4, R16, U3G, U4G

Commit message: First pass at some docs
Parts:
- C4: value 10uF 6.3V -> 10uF 10V; Comment (none) -> Optional, 3.3V bulk for SD card
- C5: Comment (none) -> Optional, 5V bulk for board
- D4: Comment (none) -> 1N5818 or 1N5819 also works
- H1, H2, H3, H4: value MountingHole -> M3 Mounting Hole
- J1: Comment (none) -> No Pin 12, Pin 13 SIO = Pin 12 on header
- J10: Comment (none) -> Do not connect Pin 12 in cable
- J2: Comment (none) -> Optional, Button A header
- J3: Comment (none) -> For Aliexpress MicroSD module if not using SMD footprint
- J4: Comment (none) -> Optional, Button B header
- J5: Comment (none) -> Optional, Reset button header
- J6: Comment (none) -> Optional, Wifi LED header
- J7: Comment (none) -> Optional, SIO LED header
- J8: Comment (none) -> Optional, Bluetooth LED header
- R1: Comment (none) -> For WiFi LED
- R10, R11, R12, R13: Comment (none) -> Optional, pull-up when using SMD SD connector
- R14, R15: Comment (none) -> Optional, only used to show SIO voltage in web UI
- R2: Comment (none) -> For SIO LED
- R3: Comment (none) -> For bluetooth LED
Changed lines of the file:
@@
 F 2 "Resistor_THT:R_Axial_DIN0207_L6.3mm_D2.5mm_P7.62mm_Horizontal" V 3430 5550 50  0001 C CNN
 F 3 "~" H 3500 5550 50  0001 C CNN
+F 4 "For WiFi LED" V 3500 5550 50  0001 C CNN "Comment"
 	1    3500 5550
 	0    1    1    0
@@
 F 2 "Resistor_THT:R_Axial_DIN0207_L6.3mm_D2.5mm_P7.62mm_Horizontal" V 3480 6250 50  0001 C CNN
 F 3 "~" H 3550 6250 50  0001 C CNN
+F 4 "For SIO LED" V 3550 6250 50  0001 C CNN "Comment"
 	1    3550 6250
 	0    1    1    0
@@
 F 2 "Resistor_THT:R_Axial_DIN0207_L6.3mm_D2.5mm_P7.62mm_Horizontal" V 3480 6950 50  0001 C CNN
 F 3 "~" H 3550 6950 50  0001 C CNN
+F 4 "For bluetooth LED" V 3550 6950 50  0001 C CNN "Comment"
 	1    3550 6950
 	0    1    1    0
@@
 F 2 "Connector_PinHeader_2.54mm:PinHeader_1x12_P2.54mm_Vertical" H 950 1700 50  0001 C CNN
 F 3 "~" H 950 1700 50  0001 C CNN
+F 4 "No Pin 12, Pin 13 SIO = Pin 12 on header" H 950 1700 50  0001 C CNN "Comment"
 	1    950  1700
 	-1   0    0    1
@@
 F 2 "Resistor_THT:R_Axial_DIN0207_L6.3mm_D2.5mm_P7.62mm_Horizontal" V 7980 4650 50  0001 C CNN
 F 3 "~" H 8050 4650 50  0001 C CNN
+F 4 "Optional, pull-up when using SMD SD connector" H 8050 4650 50  0001 C CNN "Comment"
 	1    8050 4650
 	-1   0    0    1
@@
 F 2 "Resistor_THT:R_Axial_DIN0207_L6.3mm_D2.5mm_P7.62mm_Horizontal" V 8280 4650 50  0001 C CNN
 F 3 "~" H 8350 4650 50  0001 C CNN
+F 4 "Optional, pull-up when using SMD SD connector" H 8350 4650 50  0001 C CNN "Comment"
 	1    8350 4650
 	-1   0    0    1
@@
 F 2 "Resistor_THT:R_Axial_DIN0207_L6.3mm_D2.5mm_P7.62mm_Horizontal" V 8580 4650 50  0001 C CNN
 F 3 "~" H 8650 4650 50  0001 C CNN
+F 4 "Optional, pull-up when using SMD SD connector" H 8650 4650 50  0001 C CNN "Comment"
 	1    8650 4650
 	-1   0    0    1
@@
 F 2 "Resistor_THT:R_Axial_DIN0207_L6.3mm_D2.5mm_P7.62mm_Horizontal" V 8880 4650 50  0001 C CNN
 F 3 "~" H 8950 4650 50  0001 C CNN
+F 4 "Optional, pull-up when using SMD SD connector" H 8950 4650 50  0001 C CNN "Comment"
 	1    8950 4650
 	-1   0    0    1
@@
 F 2 "Connector_PinHeader_2.54mm:PinHeader_1x06_P2.54mm_Vertical" H 10150 3550 50  0001 C CNN
 F 3 "~" H 10150 3550 50  0001 C CNN
+F 4 "For Aliexpress MicroSD module if not using SMD footprint" H 10150 3550 50  0001 C CNN "Comment"
 	1    10150 3550
 	1    0    0    -1
@@
 F 2 "Resistor_THT:R_Axial_DIN0207_L6.3mm_D2.5mm_P7.62mm_Horizontal" V 9480 2400 50  0001 C CNN
 F 3 "~" H 9550 2400 50  0001 C CNN
+F 4 "Optional, only used to show SIO voltage in web UI" H 9550 2400 50  0001 C CNN "Comment"
 	1    9550 2400
 	-1   0    0    1
@@
 F 2 "Resistor_THT:R_Axial_DIN0207_L6.3mm_D2.5mm_P7.62mm_Horizontal" V 9480 2700 50  0001 C CNN
 F 3 "~" H 9550 2700 50  0001 C CNN
+F 4 "Optional, only used to show SIO voltage in web UI" H 9550 2700 50  0001 C CNN "Comment"
 	1    9550 2700
 	-1   0    0    1
@@
 P 6150 6900
 F 0 "H1" H 6250 6946 50  0000 L CNN
-F 1 "MountingHole" H 6250 6855 50  0000 L CNN
+F 1 "M3 Mounting Hole" H 6250 6855 50  0000 L CNN
 F 2 "MountingHole:MountingHole_3.2mm_M3" H 6150 6900 50  0001 C CNN
 F 3 "~" H 6150 6900 50  0001 C CNN
@@
 P 6150 7100
 F 0 "H2" H 6250 7146 50  0000 L CNN
-F 1 "MountingHole" H 6250 7055 50  0000 L CNN
+F 1 "M3 Mounting Hole" H 6250 7055 50  0000 L CNN
 F 2 "MountingHole:MountingHole_3.2mm_M3" H 6150 7100 50  0001 C CNN
 F 3 "~" H 6150 7100 50  0001 C CNN
@@
 P 6150 7300
 F 0 "H3" H 6250 7346 50  0000 L CNN
-F 1 "MountingHole" H 6250 7255 50  0000 L CNN
+F 1 "M3 Mounting Hole" H 6250 7255 50  0000 L CNN
 F 2 "MountingHole:MountingHole_3.2mm_M3" H 6150 7300 50  0001 C CNN
 F 3 "~" H 6150 7300 50  0001 C CNN
@@
 P 6150 7500
 F 0 "H4" H 6250 7546 50  0000 L CNN
-F 1 "MountingHole" H 6250 7455 50  0000 L CNN
+F 1 "M3 Mounting Hole" H 6250 7455 50  0000 L CNN
 F 2 "MountingHole:MountingHole_3.2mm_M3" H 6150 7500 50  0001 C CNN
 F 3 "~" H 6150 7500 50  0001 C CNN
@@
 F 2 "Connector_PinHeader_2.54mm:PinHeader_1x02_P2.54mm_Vertical" H 6000 4300 50  0001 C CNN
 F 3 "~" H 6000 4300 50  0001 C CNN
+F 4 "Optional, Button A header" V 6000 4300 50  0001 C CNN "Comment"
 	1    6000 4300
 	0    1    1    0
@@
 F 2 "Connector_PinHeader_2.54mm:PinHeader_1x02_P2.54mm_Vertical" H 6000 5000 50  0001 C CNN
 F 3 "~" H 6000 5000 50  0001 C CNN
+F 4 "Optional, Button B header" V 6000 5000 50  0001 C CNN "Comment"
 	1    6000 5000
 	0    1    1    0
@@
 F 2 "Connector_PinHeader_2.54mm:PinHeader_1x02_P2.54mm_Vertical" H 6000 5750 50  0001 C CNN
 F 3 "~" H 6000 5750 50  0001 C CNN
+F 4 "Optional, Reset button header" V 6000 5750 50  0001 C CNN "Comment"
 	1    6000 5750
 	0    1    1    0
@@
 F 2 "Connector_PinHeader_2.54mm:PinHeader_1x02_P2.54mm_Vertical" H 4100 5900 50  0001 C CNN
 F 3 "~" H 4100 5900 50  0001 C CNN
+F 4 "Optional, Wifi LED header" V 4100 5900 50  0001 C CNN "Comment"
 	1    4100 5900
 	0    1    1    0
@@
 F 2 "Connector_PinHeader_2.54mm:PinHeader_1x02_P2.54mm_Vertical" H 4100 6600 50  0001 C CNN
 F 3 "~" H 4100 6600 50  0001 C CNN
+F 4 "Optional, SIO LED header" V 4100 6600 50  0001 C CNN "Comment"
 	1    4100 6600
 	0    1    1    0
@@
 F 2 "Connector_PinHeader_2.54mm:PinHeader_1x02_P2.54mm_Vertical" H 4100 7300 50  0001 C CNN
 F 3 "~" H 4100 7300 50  0001 C CNN
+F 4 "Optional, Bluetooth LED header" V 4100 7300 50  0001 C CNN "Comment"
 	1    4100 7300
 	0    1    1    0
@@
 P 8650 3550
 F 0 "C4" H 8765 3596 50  0000 L CNN
-F 1 "10uF 6.3V" H 8765 3505 50  0000 L CNN
+F 1 "10uF 10V" H 8765 3505 50  0000 L CNN
 F 2 "Capacitor_THT:CP_Radial_Tantal_D5.5mm_P5.00mm" H 8650 3550 50  0001 C CNN
 F 3 "~" H 8650 3550 50  0001 C CNN
+F 4 "Optional, 3.3V bulk for SD card" H 8650 3550 50  0001 C CNN "Comment"
 	1    8650 3550
 	1    0    0    -1
@@
 F 2 "Connector_Dsub:DSUB-15_Female_Horizontal_P2.77x2.84mm_EdgePinOffset4.94mm_Housed_MountingHolesOffset7.48mm" H 1650 3600 50  0001 C CNN
 F 3 " ~" H 1650 3600 50  0001 C CNN
+F 4 "Do not connect Pin 12 in cable" H 1650 3600 50  0001 C CNN "Comment"
 	1    1650 3600
 	1    0    0    -1
@@
 F 2 "Diode_THT:D_DO-41_SOD81_P10.16mm_Horizontal" H 1650 4975 50  0001 C CNN
 F 3 "http://www.vishay.com/docs/88525/1n5817.pdf" H 1650 5150 50  0001 C CNN
+F 4 "1N5818 or 1N5819 also works" H 1650 5150 50  0001 C CNN "Comment"
 	1    1650 5150
 	-1   0    0    1
@@
 F 2 "Capacitor_THT:CP_Radial_D6.3mm_P2.50mm" H 1750 5950 50  0001 C CNN
 F 3 "~" H 1750 5950 50  0001 C CNN
+F 4 "Optional, 5V bulk for board" V 1750 5950 50  0001 C CNN "Comment"
 	1    1750 5950
 	1    0    0    -1
